File: prototipo_1/placa_smd_kgf1.kicad_pcb (KiCad board)
At the start: 2 copper layers, 12 parts

Commit message: Actualizacion de prototipo
Parts:
- removed REF** (x5): TestPoint_Pad_4.0x4.0mm, TestPoint:TestPoint_Pad_4.0x4.0mm
- removed REF** (x5): R_2512_6332Metric, Resistor_SMD:R_2512_6332Metric
- removed REF** (x2): D_SMB, Diode_SMD:D_SMB
- added D1: D, Diode_SMD:D_SMB-SMC_Universal_Handsoldering, F.Cu at (125.0, 80.0)
- added D2: D, Diode_SMD:D_SMB-SMC_Universal_Handsoldering, F.Cu at (135.0, 82.0)
- added J1: Conn_01x01_Female, Connector_PinHeader_2.54mm:PinHeader_1x01_P2.54mm_Vertical, F.Cu at (125.0, 100.0)
- added J2: Conn_01x03_Female, Connector_PinHeader_2.54mm:PinHeader_1x03_P2.54mm_Vertical, F.Cu at (133.0, 76.5)
- added J3: Conn_01x01_Female, Connector_PinHeader_2.54mm:PinHeader_1x01_P2.54mm_Vertical, F.Cu at (145.0, 84.0)
- added R1: 22R, Resistor_SMD:R_2512_6332Metric_Pad1.52x3.35mm_HandSolder, F.Cu at (125.0, 92.0)
- added R2: 22R, Resistor_SMD:R_2512_6332Metric_Pad1.52x3.35mm_HandSolder, F.Cu at (130.0, 92.0)
- added R3: 22R, Resistor_SMD:R_2512_6332Metric_Pad1.52x3.35mm_HandSolder, F.Cu at (135.0, 92.0)
- added R4: 22R, Resistor_SMD:R_2512_6332Metric_Pad1.52x3.35mm_HandSolder, F.Cu at (140.0, 92.0)
- added R5: 22R, Resistor_SMD:R_2512_6332Metric_Pad1.52x3.35mm_HandSolder, F.Cu at (145.0, 92.0)
Routing:
- net (no net): track 94.2 -> 0.00 mm
Other:
- board outline added: 30 x 35 mm
- rule pad_to_mask_clearance: 0.051 -> 0

Commit message: Actualizacion de prototipo
Parts:
- moved R5 19.6 mm to (125.5, 90.0), turned to 0 degrees
- moved R1 18.0 mm to (125.5, 110.0), turned to 0 degrees
- moved R4 14.8 mm to (125.5, 95.0), turned to 0 degrees
- moved J3 13.9 mm to (132.5, 90.0)
- moved R2 13.8 mm to (125.5, 105.0), turned to 0 degrees
- moved J1 12.5 mm to (132.5, 110.0)
- moved R3 12.4 mm to (125.5, 100.0), turned to 0 degrees
- moved J2 9.18 mm to (125.0, 72.0)
- moved D2 3.20 mm to (132.5, 80.0), turned to 270 degrees
- moved D1 1.00 mm to (124.0, 80.0)
Other:
- board size 30 x 35 mm -> 15 x 42.5 mm
